File: v2.0-typec-CH340X/Watchy.kicad_sch (KiCad schematic)
At the start: 61 parts, among them J1 FPC24(0.5MM), J2 Conn_01x04, J3 Battery, J4 Conn_01x04, M1 Vibration_Motor, Q1 AO3400A, Q4 CJ2301, Q5 S8050, SW1 BTN, SW2 BTN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

Commit message: add schema pdf files
Other:
- note removed: "1=charging 当没有电池时, VBUS 5v变成VBAT VBAT: 4.2v 此时时钟有问题, 可能是换了TP4057导致 当没有电池时, VBAT: 3.75v"
Changed lines of the file:
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@@
-		)
-	)
-	(text "1=charging\n当没有电池时, VBUS 5v变成VBAT\nVBAT: 4.2v 此时时钟有问题, 可能是换了TP4057导致\n当没有电池时, VBAT: 3.75v"
-		(exclude_from_sim no)
-		(at 34.544 141.986 0)
-		(effects
-			(font
-				(size 1.016 1.016)
-			)
-			(justify left)
 		)
 	)
